File: rf.kicad_sch (KiCad schematic)
At the start: 9 parts, among them U3 E22-900M30S, U4 E22-400M30S

Commit message: Updated schematic and pcb for rf
Parts:
- removed ANT2: 400MHz SMA, Connector_Coaxial:SMA_Molex_73251-1153_EdgeMount_Horizontal, symbol Connector:Conn_Coaxial
- removed C14: 0.1u, Capacitor_SMD:C_0603_1608Metric, symbol Device:C
- removed C15: 1u, Capacitor_SMD:C_0603_1608Metric, symbol Device:C
- removed U4: E22-400M30S, LEOS:XCVR_E22-900M30S, symbol LEOS:E22-400M30S
Connections:
- net at U3.7 (TXEN), U3.8 (DIO2): no longer U3.6 (RXEN)
- new net RXEN: U3.6 (RXEN)
Other:
- moved on the sheet: ANT1, C12, C13, R2, U3
