File: LEOS-radio.kicad_pcb (KiCad board)
At the start: 2 copper layers, 100.1 x 100 mm, 31 parts, among them J1 MicroFit_1x4, J2 MicroFit_1x4, U1 MCP2562FD, U2 MCP2518FD, U3 E22-900M30S, U4 E22-400M30S, Y1 40 MHz

Commit message: Updated schematic and pcb for rf
Parts:
- removed ANT2: 400MHz SMA, Connector_Coaxial:SMA_Molex_73251-1153_EdgeMount_Horizontal
- removed C14: 0.1u, Capacitor_SMD:C_0603_1608Metric
- removed C15: 1u, Capacitor_SMD:C_0603_1608Metric
- removed U4: E22-400M30S, LEOS:XCVR_E22-900M30S
Connections:
- A1 pad 19: /RF/CS1 -> /CS1
- A1 pad 21: /RF/INT1 -> /INT1
- A1 pad 24: /RF/BUSY1 -> /BUSY1
- A1 pad 26: unconnected-(A1-GPIO20-Pad26) -> /RF/RXEN
- U3 pad 6: Net-(U3-DIO2) -> /RF/RXEN
Routing:
- net /RF/CS1: track 102.5 -> 0.00 mm, vias 2 -> 0
- net /RF/BUSY1: track 75.2 -> 0.00 mm, vias 2 -> 0
- net /CS1: track 0.00 -> 70.5 mm, vias 0 -> 1
- net /RF/INT1: track 69.9 -> 0.00 mm, vias 2 -> 0
- net /RF/SCK: track 90.2 -> 57.2 mm, vias 2 -> 1
- net /RF/MOSI: track 90.2 -> 57.2 mm, vias 2 -> 1
- net /RF/MISO: track 90.4 -> 57.4 mm, vias 2 -> 1
- net /RF/nRESET: track 90.6 -> 57.7 mm, vias 2 -> 1
- net /RF/RF_400MHz: track 27.8 -> 0.00 mm
- net /BUSY1: track 0.00 -> 15.4 mm, vias 0 -> 1
- net /RF/RXEN: track 0.00 -> 12.2 mm
- net +5V: track 181.1 -> 171.8 mm
- net /INT1: track 0.00 -> 8.37 mm, vias 0 -> 1
- net Net-(U4-DIO2): track 5.08 -> 0.00 mm
- net Net-(U3-DIO2): track 5.08 -> 2.54 mm
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Other:
- board text removed: "433-470MHz 30 dBm 50Ω"

Commit message: updates from radio removal
Connections:
- A1 pad 19: /CS1 -> unconnected-(A1-GPIO14-Pad19)
- A1 pad 21: /INT1 -> unconnected-(A1-GPIO16-Pad21)
- A1 pad 24: /BUSY1 -> unconnected-(A1-GPIO18-Pad24)
Routing:
- net unconnected-(A1-GPIO14-Pad19): track 0.00 -> 70.5 mm, vias 0 -> 1
- net /CS1: track 70.5 -> 0.00 mm, vias 1 -> 0
- net unconnected-(A1-GPIO18-Pad24): track 0.00 -> 15.4 mm, vias 0 -> 1
- net /BUSY1: track 15.4 -> 0.00 mm, vias 1 -> 0
- net unconnected-(A1-GPIO16-Pad21): track 0.00 -> 8.37 mm, vias 0 -> 1
- net /INT1: track 8.37 -> 0.00 mm, vias 1 -> 0
