File: LEOS-radio.kicad_sch (KiCad schematic)
At the start: 3 parts

Commit message: Updated schematic and pcb for rf
Connections:
- net RF/RXEN: now reaches A1.26 (GPIO20)
- no-connect marks 16 -> 15
Other:
- sheet RF ports: added RXEN; removed none

Commit message: updates from radio removal
Connections:
- net RF/BUSY1: no longer names the net of A1.24 (GPIO18)
- net RF/CS1: no longer names the net of A1.19 (GPIO14)
- net RF/INT1: no longer names the net of A1.21 (GPIO16)
- no-connect marks 15 -> 18
Other:
- sheet RF ports: added none; removed BUSY1, CS1, INT1
Changed lines of the file:
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@@
+	)
+	(no_connect
+		(at 170.18 96.52)
 	)
 	(no_connect
@@
 	)
 	(no_connect
+		(at 170.18 91.44)
+	)
+	(no_connect
 		(at 170.18 104.14)
 	)
@@
 		(at 170.18 111.76)
 	)
+	(no_connect
+		(at 124.46 124.46)
+	)
 	(wire
 		(pts
@@
 	(wire
 		(pts
-			(xy 177.8 96.52) (xy 170.18 96.52)
-		)
-		(stroke
-			(width 0)
-			(type default)
-		)
-	)
-	(wire
-		(pts
-			(xy 97.79 137.16) (xy 97.79 158.75)
-		)
-		(stroke
-			(width 0)
-			(type default)
-		)
-	)
-	(wire
-		(pts
 			(xy 105.41 151.13) (xy 175.26 151.13)
 		)
@@
 	(wire
 		(pts
-			(xy 95.25 137.16) (xy 97.79 137.16)
-		)
-		(stroke
-			(width 0)
-			(type default)
-		)
-	)
-	(wire
-		(pts
 			(xy 95.25 114.3) (xy 124.46 114.3)
 		)
@@
 	(wire
 		(pts
-			(xy 102.87 153.67) (xy 177.8 153.67)
-		)
-		(stroke
-			(width 0)
-			(type default)
-		)
-	)
-	(wire
-		(pts
 			(xy 95.25 119.38) (xy 124.46 119.38)
 		)
@@
 	(wire
 		(pts
-			(xy 102.87 132.08) (xy 102.87 153.67)
-		)
-		(stroke
-			(width 0)
-			(type default)
-		)
-	)
-	(wire
-		(pts
 			(xy 142.24 57.15) (xy 142.24 66.04)
 		)
@@
 	(wire
 		(pts
-			(xy 95.25 132.08) (xy 102.87 132.08)
-		)
-		(stroke
-			(width 0)
-			(type default)
-		)
-	)
-	(wire
-		(pts
-			(xy 182.88 158.75) (xy 182.88 91.44)
-		)
-		(stroke
-			(width 0)
-			(type default)
-		)
-	)
-	(wire
-		(pts
 			(xy 95.25 127) (xy 124.46 127)
 		)
@@
 	(wire
 		(pts
-			(xy 182.88 91.44) (xy 170.18 91.44)
-		)
-		(stroke
-			(width 0)
-			(type default)
-		)
-	)
-	(wire
-		(pts
 			(xy 95.25 116.84) (xy 124.46 116.84)
 		)
@@
 	(wire
 		(pts
-			(xy 97.79 158.75) (xy 182.88 158.75)
-		)
-		(stroke
-			(width 0)
-			(type default)
-		)
-	)
-	(wire
-		(pts
 			(xy 95.25 121.92) (xy 124.46 121.92)
 		)
@@
 	(wire
 		(pts
-			(xy 177.8 153.67) (xy 177.8 96.52)
-		)
-		(stroke
-			(width 0)
-			(type default)
-		)
-	)
-	(wire
-		(pts
 			(xy 95.25 93.98) (xy 124.46 93.98)
-		)
-		(stroke
-			(width 0)
-			(type default)
-		)
-	)
-	(wire
-		(pts
-			(xy 95.25 124.46) (xy 124.46 124.46)
 		)
 		(stroke
@@
 			)
 		)
-		(pin "CS1" input
-			(at 95.25 124.46 0)
-			(effects
-				(font
-					(size 1.27 1.27)
-				)
-				(justify right)
-			)
-		)
 		(pin "MISO" output
 			(at 95.25 119.38 0)
@@
 			)
 		)
-		(pin "BUSY1" input
-			(at 95.25 132.08 0)
-			(effects
-				(font
-					(size 1.27 1.27)
-				)
-				(justify right)
-			)
-		)
 		(pin "INT0" input
 			(at 95.25 134.62 0)
 			(effects
 				(font
-					(size 1.27 1.27)
-				)
-				(justify right)
-			)
-		)
-		(pin "INT1" input
-			(at 95.25 137.16 0)
-			(effects
-				(font
