File: connectors.kicad_sch (KiCad schematic)
At the start: 7 parts, among them J1 MicroFit_1x4, J2 MicroFit_1x4

Commit message: updates from radio removal
Parts:
- R1: Digikey CF14JT120RCT-ND -> 13-CFR-25JR-52-120RCT-ND; MPN CF14JT120R -> CFR-25JR-52-120R; Manufacturer Stackpole Electronics Inc -> YAGEO
